File: single_motor_driver/single_motor_driver_v6.brd (EAGLE design)
At the start: 100 x 80 mm, 44 parts, among them IC1 MCP602SN

Commit message: last version finished, pls work!
Parts:
- removed IC1: MCP602SN, dedo:SO08
- removed J1, J2: (no value), uchile_robotics_eagle_lib:1X02
- removed RF1, RF2: 200k, resistor:R0805
- removed RF3: 10k, resistor:R0805
- removed RF4: 1k, resistor:R0805
- added ZERO: 0, resistor:R0805
- moved RL10 122.2 mm to (51.3, 18.0), flipped to the bottom, turned to 180 degrees
- moved RF7 119.8 mm to (50.8, 38.4), flipped to the bottom, turned to 180 degrees
- moved RF6 114.5 mm to (50.8, 40.9), flipped to the bottom, turned to 180 degrees
- moved RF5 109.9 mm to (50.8, 35.8), flipped to the bottom, turned to 180 degrees
- moved CVDD2 108.9 mm to (58.7, 23.1), flipped to the bottom, turned to 180 degrees
- moved LED4 107.7 mm to (54.9, 3.56), turned to 180 degrees
- moved RGHA2 101.6 mm to (33.0, 29.5), turned to 180 degrees
- moved LED3 97.0 mm to (58.9, 31.5), turned to 180 degrees
- moved RL5 92.9 mm to (31.8, 11.2), turned to 90 degrees
- moved RL6 92.8 mm to (27.7, 18.8)
- moved RL9 81.8 mm to (50.8, 28.2), flipped to the bottom, turned to 180 degrees
- moved RL11 79.7 mm to (58.9, 26.7), turned to 270 degrees
- moved RL3 77.6 mm to (31.8, 21.8), turned to 90 degrees
- moved RL4 77.2 mm to (26.7, 29.5)
- moved RL8 76.2 mm to (50.8, 30.7), flipped to the bottom, turned to 180 degrees
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Connections:
- removed net -5V: RF3.1, U$3.2
- removed net GND1: C1.-, C3.-, CVDD1.2
- removed net GND2: U$2.VREG
- removed net N$52: IC1.2, J1.2, RF1.1
- removed net N$82: IC1.6, J2.2, RF2.2
- removed net VOUT1: IC1.1, RF1.2, U$1.7
- removed net VOUT2: IC1.7, RF2.1
- removed net VT: J1.1, J2.1, RF3.2, RF4.1
- new net LSS: A.1, B.1, C.1, RL1.1, RL3.1, RL5.1, U$2.LSS
- new net PGND: C1.-, C3.-, CVDD1.2, RF11.2, U$3.1, U$3.2, ZERO.2
- net +24V: now also U$3.3
- net +5V: now also U$1.7; no longer IC1.8, U$3.3
- net GND: now also U$2.VREG, ZERO.1; no longer A.1, B.1, C.1, IC1.3, IC1.4, IC1.5, RF11.2, RF4.2, RL1.1, RL3.1, RL5.1, U$2.LSS, U$3.1
Routing:
- net GND: track 0.00 -> 185.8 mm, vias 0 -> 4
- net +5V: track 0.00 -> 137.2 mm, vias 0 -> 1
- net +24V: track 0.00 -> 135.5 mm, vias 0 -> 4
- net PGND: track 0.00 -> 134.2 mm, vias 0 -> 4
- net HB: track 0.00 -> 116.4 mm, vias 0 -> 3
- net HA: track 0.00 -> 109.5 mm, vias 0 -> 3
- net HC: track 0.00 -> 96.3 mm, vias 0 -> 3
- net LSS: track 0.00 -> 67.0 mm, vias 0 -> 4
- net MOTOR_1: track 29.8 -> 74.3 mm, vias 0 -> 1
- net MOTOR_3: track 29.0 -> 68.2 mm, vias 0 -> 1
- net N$17: track 0.00 -> 36.3 mm, vias 0 -> 1
- net BRAKEN: track 0.00 -> 31.7 mm, vias 0 -> 1
- net N$27: track 0.00 -> 29.6 mm, vias 0 -> 1
- net ENABLE: track 0.00 -> 29.5 mm, vias 0 -> 1
- net MOTOR_2: track 23.2 -> 52.7 mm, vias 0 -> 1
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- added copper zone on layer 1, net GND
- added copper zone on layer 16, net GND
- added copper zone on layer 16, net N$3
- added copper zone on layer 1, net PGND
Other:
- board size 100 x 80 mm -> 61.9 x 49.5 mm

Commit message: last update, working
Parts:
- moved ZERO 2.29 mm to (24.1, 42.7)
- moved U$3 1.02 mm to (20.3, 46.7)
Connections:
- removed net LSS: A.1, B.1, C.1, RL1.1, RL3.1, RL5.1, U$2.LSS
- net PGND: now also A.1, B.1, C.1, RL1.1, RL3.1, RL5.1, U$2.LSS
Routing:
- net PGND: track 134.2 -> 221.6 mm, vias 4 -> 8
- net LSS: track 67.0 -> 0.00 mm, vias 4 -> 0
- net MOTOR_1: track 74.3 -> 72.8 mm
- net GND: track 185.8 -> 184.9 mm
- added copper zone on layer 16, net PGND
- removed copper zone on layer 16, net N$3
