File: single_motor_driver/single_motor_driver_v6.sch (EAGLE design)
At the start: 44 parts, among them IC1 MCP602SN

Commit message: last version finished, pls work!
Parts:
- removed IC1: MCP602SN, dedo:MCP602SN
- removed J1, J2: (no value), uchile_robotics_eagle_lib:M02PTH
- removed RF1, RF2: 200k, resistor:R-US_R0805
- removed RF3: 10k, resistor:R-US_R0805
- removed RF4: 1k, resistor:R-US_R0805
- added ZERO: 0, resistor:R-US_R0805
Connections:
- removed net -5V: RF3.1, U$3.VDD
- removed net GND1: C1.-, C3.-, CVDD1.2
- removed net GND2: U$2.VREG
- removed net N$52: IC1A.-IN, J1.2, RF1.1
- removed net N$82: IC1B.-IN, J2.2, RF2.2
- removed net VOUT1: IC1A.OUT, RF1.2, U$17.S
- removed net VOUT2: IC1B.OUT, RF2.1
- removed net VT: J1.1, J2.1, RF3.2, RF4.1
- new net LSS: A.S1, B.S1, C.S1, RL1.1, RL3.1, RL5.1, U$2.LSS
- new net PGND: C1.-, C3.-, CVDD1.2, RF11.2, U$3.GND, U$3.VDD, ZERO.2
- net +24V: now also U$3.D+
- net +5V: now also U$17.S; no longer IC1P.V+, U$3.D+
- net GND: now also U$2.VREG, ZERO.1; no longer A.S1, B.S1, C.S1, IC1A.+IN, IC1B.+IN, IC1P.V-, RF11.2, RF4.2, RL1.1, RL3.1, RL5.1, U$2.LSS, U$3.GND
Other:
- moved on the sheet: LED2, LED4, RF11, RF12

Commit message: last update, working
Connections:
- removed net LSS: A.S1, B.S1, C.S1, RL1.1, RL3.1, RL5.1, U$2.LSS
- net PGND: now also A.S1, B.S1, C.S1, RL1.1, RL3.1, RL5.1, U$2.LSS
Changed lines of the file:
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@@
 <part name="SUPPLY8" library="supply2" library_urn="urn:adsk.eagle:library:372" deviceset="GND1" device=""/>
 <part name="SUPPLY9" library="supply2" library_urn="urn:adsk.eagle:library:372" deviceset="GND" device=""/>
+<part name="SUPPLY12" library="supply2" library_urn="urn:adsk.eagle:library:372" deviceset="GND1" device=""/>
 </parts>
 <sheets>
@@
 <instance part="SUPPLY8" gate="G$1" x="-7.62" y="48.26"/>
 <instance part="SUPPLY9" gate="GND" x="12.7" y="48.26"/>
+<instance part="SUPPLY12" gate="G$1" x="-38.1" y="35.56"/>
 </instances>
 <busses>
@@
 </segment>
 </net>
-<net name="LSS" class="0">
+<net name="PGND" class="0">
+<segment>
+<pinref part="C3" gate="G$1" pin="-"/>
+<pinref part="SUPPLY10" gate="G$1" pin="GND1"/>
+<wire x1="-101.6" y1="106.68" x2="-101.6" y2="111.76" width="0.1524" layer="91"/>
+</segment>
+<segment>
+<pinref part="C1" gate="G$1" pin="-"/>
+<pinref part="SUPPLY3" gate="G$1" pin="GND1"/>
+<wire x1="-101.6" y1="33.02" x2="-101.6" y2="35.56" width="0.1524" layer="91"/>
+</segment>
+<segment>
+<pinref part="CVDD1" gate="G$1" pin="2"/>
+<pinref part="SUPPLY2" gate="G$1" pin="GND1"/>
+</segment>
+<segment>
+<pinref part="U$3" gate="J$1" pin="GND"/>
+<pinref part="SUPPLY6" gate="G$1" pin="GND1"/>
+<wire x1="25.4" y1="22.86" x2="33.02" y2="22.86" width="0.1524" layer="91"/>
+<pinref part="U$3" gate="J$1" pin="VDD"/>
+<wire x1="33.02" y1="25.4" x2="25.4" y2="25.4" width="0.1524" layer="91"/>
+<wire x1="25.4" y1="25.4" x2="25.4" y2="22.86" width="0.1524" layer="91"/>
+<pinref part="RF11" gate="G$1" pin="2"/>
+<wire x1="17.78" y1="22.86" x2="25.4" y2="22.86" width="0.1524" layer="91"/>
+<junction x="25.4" y="22.86"/>
+</segment>
+<segment>
+<pinref part="ZERO" gate="G$1" pin="2"/>
+<pinref part="SUPPLY8" gate="G$1" pin="GND1"/>
+<wire x1="-7.62" y1="50.8" x2="-2.54" y2="50.8" width="0.1524" layer="91"/>
+</segment>
 <segment>
 <pinref part="C" gate="G$1" pin="S1"/>
@@
 <wire x1="-10.16" y1="101.6" x2="-38.1" y2="101.6" width="0.1524" layer="91"/>
 <junction x="-38.1" y="101.6"/>
-</segment>
-</net>
-<net name="PGND" class="0">
-<segment>
-<pinref part="C3" gate="G$1" pin="-"/>
-<pinref part="SUPPLY10" gate="G$1" pin="GND1"/>
-<wire x1="-101.6" y1="106.68" x2="-101.6" y2="111.76" width="0.1524" layer="91"/>
-</segment>
-<segment>
-<pinref part="C1" gate="G$1" pin="-"/>
-<pinref part="SUPPLY3" gate="G$1" pin="GND1"/>
-<wire x1="-101.6" y1="33.02" x2="-101.6" y2="35.56" width="0.1524" layer="91"/>
-</segment>
-<segment>
-<pinref part="CVDD1" gate="G$1" pin="2"/>
-<pinref part="SUPPLY2" gate="G$1" pin="GND1"/>
-</segment>
-<segment>
-<pinref part="U$3" gate="J$1" pin="GND"/>
-<pinref part="SUPPLY6" gate="G$1" pin="GND1"/>
-<wire x1="25.4" y1="22.86" x2="33.02" y2="22.86" width="0.1524" layer="91"/>
-<pinref part="U$3" gate="J$1" pin="VDD"/>
-<wire x1="33.02" y1="25.4" x2="25.4" y2="25.4" width="0.1524" layer="91"/>
-<wire x1="25.4" y1="25.4" x2="25.4" y2="22.86" width="0.1524" layer="91"/>
-<pinref part="RF11" gate="G$1" pin="2"/>
-<wire x1="17.78" y1="22.86" x2="25.4" y2="22.86" width="0.1524" layer="91"/>
-<junction x="25.4" y="22.86"/>
-</segment>
-<segment>
-<pinref part="ZERO" gate="G$1" pin="2"/>
-<pinref part="SUPPLY8" gate="G$1" pin="GND1"/>
-<wire x1="-7.62" y1="50.8" x2="-2.54" y2="50.8" width="0.1524" layer="91"/>
-</segment>
-</net>
+<pinref part="SUPPLY12" gate="G$1" pin="GND1"/>
+<junction x="-38.1" y="38.1"/>
+</segment>
+</net>
