File: tssop28breakout/tssop28breakout.brd (EAGLE design)
At the start: 17.8 x 33 mm, 8 parts

Commit message: last version finished, pls work!
Parts:
- moved C5 8.84 mm to (7.62, 9.53), turned to 270 degrees
- moved C4 2.29 mm to (12.1, 10.2)
Connections:
- new net PAD: U$1.PAD
- net GND: no longer U$1.PAD
Routing:
- net N$28: track 4.77 -> 16.2 mm
- net N$14: track 12.7 -> 2.25 mm
- net GND: track 24.0 -> 17.2 mm
- net N$27: track 5.75 -> 3.80 mm
- net N$26: track 6.45 -> 4.55 mm
Changed lines of the file:
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@@
 <setting verticaltext="up"/>
 </settings>
-<grid distance="25" unitdist="mil" unit="mm" style="lines" multiple="1" display="yes" altdistance="2.5" altunitdist="mil" altunit="mm"/>
+<grid distance="10" unitdist="mil" unit="mil" style="lines" multiple="1" display="yes" altdistance="2.5" altunitdist="mil" altunit="mm"/>
 <layers>
 <layer number="1" name="Top" color="4" fill="1" visible="yes" active="yes"/>
@@
 <dimension x1="-1.27" y1="1.27" x2="-1.27" y2="31.75" x3="-5.08" y3="16.51" textsize="1.778" layer="1"/>
 <dimension x1="1.27" y1="34.925" x2="16.51" y2="34.925" x3="8.89" y3="38.1" textsize="1.778" layer="1"/>
+<rectangle x1="10.16" y1="13.97" x2="10.795" y2="15.24" layer="1"/>
+<rectangle x1="8.382" y1="14.224" x2="11.684" y2="32.512" layer="1"/>
 </plain>
 <attributes>
@@
 <element name="U$1" library="dedo" package="TSSOP28" value="A9415" x="10" y="16.73" rot="R270"/>
 <element name="C3" library="resistor" package="C0805" value="0.033uF" x="5.065" y="3.795"/>
-<element name="C4" library="resistor" package="C0805" value="0.47uF" x="10.16" y="8.89" rot="R90"/>
-<element name="C5" library="resistor" package="C0805" value="0.68uF" x="10.795" y="1.27"/>
+<element name="C4" library="resistor" package="C0805" value="0.47uF" x="12.065" y="10.16" rot="R90"/>
+<element name="C5" library="resistor" package="C0805" value="0.68uF" x="7.62" y="9.525" rot="R270"/>
 <element name="C1" library="resistor" package="C0805" value="0.033uF" x="3.81" y="20.32" rot="R270"/>
 <element name="C2" library="resistor" package="C0805" value="0.033uF" x="3.175" y="15.24" rot="R270"/>
@@
 <contactref element="U$1" pad="11"/>
 <wire x1="7.0822" y1="14.455" x2="6.2" y2="14.455" width="0.4064" layer="1"/>
-<wire x1="5.08" y1="13.335" x2="5.08" y2="7.62" width="0.4064" layer="1"/>
-<wire x1="5.08" y1="7.62" x2="3.81" y2="6.35" width="0.4064" layer="1"/>
+<wire x1="4.318" y1="12.573" x2="4.318" y2="6.858" width="0.4064" layer="1"/>
+<wire x1="4.318" y1="6.858" x2="3.81" y2="6.35" width="0.4064" layer="1"/>
 <wire x1="3.81" y1="6.35" x2="1.27" y2="6.35" width="0.4064" layer="1"/>
-<wire x1="6.2" y1="14.455" x2="5.08" y2="13.335" width="0.4064" layer="1"/>
+<wire x1="6.2" y1="14.455" x2="4.318" y2="12.573" width="0.4064" layer="1"/>
 </signal>
 <signal name="N$12">
@@
 <wire x1="4.1" y1="3.81" x2="1.27" y2="3.81" width="0.4064" layer="1"/>
 <contactref element="C3" pad="1"/>
-<wire x1="6.3501375" y1="13.7138" x2="5.6725" y2="13.0361625" width="0.4064" layer="1"/>
-<wire x1="5.6725" y1="13.0361625" x2="5.6725" y2="11.9738375" width="0.4064" layer="1"/>
-<wire x1="7.0822" y1="13.805" x2="6.991" y2="13.7138" width="0.4064" layer="1"/>
-<wire x1="6.991" y1="13.7138" x2="6.3501375" y2="13.7138" width="0.4064" layer="1"/>
-<wire x1="5.6725" y1="11.9738375" x2="5.715" y2="11.9313375" width="0.4064" layer="1"/>
 <wire x1="4.1" y1="4.735" x2="4.1" y2="3.81" width="0.4064" layer="1"/>
-<wire x1="5.715" y1="11.9313375" x2="5.715" y2="6.35" width="0.4064" layer="1"/>
-<wire x1="5.715" y1="6.35" x2="4.1" y2="4.735" width="0.4064" layer="1"/>
+<wire x1="5.1645" y1="5.7995" x2="4.1" y2="4.735" width="0.4064" layer="1"/>
+<wire x1="5.1645" y1="12.5281625" x2="5.1645" y2="5.7995" width="0.4064" layer="1"/>
+<wire x1="7.0822" y1="13.805" x2="6.4413375" y2="13.805" width="0.4064" layer="1"/>
+<wire x1="6.4413375" y1="13.805" x2="5.1645" y2="12.5281625" width="0.4064" layer="1"/>
 <wire x1="4.1" y1="3.81" x2="4.115" y2="3.795" width="0" layer="19" extent="1-1"/>
 </signal>
@@
 </polygon>
 <contactref element="U$1" pad="17"/>
-<contactref element="U$1" pad="PAD"/>
-<wire x1="10.925" y1="13.805" x2="12.9178" y2="13.805" width="0.4064" layer="1"/>
-<wire x1="10.925" y1="13.805" x2="10" y2="14.73" width="0.4064" layer="1"/>
-<wire x1="10" y1="15.356321875" x2="10" y2="14.73" width="0.4064" layer="1"/>
 <contactref element="JP2" pad="2"/>
-<wire x1="10" y1="15.356321875" x2="10" y2="16.73" width="0.4064" layer="1"/>
-<wire x1="16.51" y1="3.81" x2="12.7" y2="3.81" width="0.4064" layer="1"/>
-<wire x1="12.7" y1="3.81" x2="10.16" y2="6.35" width="0.4064" layer="1"/>
-<wire x1="10.16" y1="6.35" x2="8.89" y2="6.35" width="0.4064" layer="1"/>
-<wire x1="8.89" y1="6.35" x2="8.89" y2="15.24" width="0.4064" layer="1"/>
-<wire x1="8.89" y1="15.24" x2="9.883678125" y2="15.24" width="0.4064" layer="1"/>
-<wire x1="9.883678125" y1="15.24" x2="10" y2="15.356321875" width="0.4064" layer="1"/>
+<wire x1="12.9178" y1="13.805" x2="10.16" y2="13.805" width="0.4064" layer="1"/>
+<wire x1="10.16" y1="7.62" x2="13.335" y2="7.62" width="0.4064" layer="1"/>
+<wire x1="16.51" y1="4.445" x2="16.51" y2="3.81" width="0.4064" layer="1"/>
+<wire x1="10.16" y1="13.805" x2="10.16" y2="7.62" width="0.4064" layer="1"/>
+<wire x1="13.335" y1="7.62" x2="16.51" y2="4.445" width="0.4064" layer="1"/>
 </signal>
 <signal name="N$26">
 <contactref element="U$1" pad="15"/>
 <contactref element="C4" pad="1"/>
-<wire x1="12.32729375" y1="8.8344" x2="12.3244" y2="8.8344" width="0.4064" layer="1"/>
-<wire x1="12.9178" y1="12.505" x2="12.9178" y2="9.42490625" width="0.4064" layer="1"/>
-<wire x1="12.9178" y1="9.42490625" x2="12.32729375" y2="8.8344" width="0.4064" layer="1"/>
-<wire x1="12.3244" y1="8.8344" x2="11.43" y2="7.94" width="0.4064" layer="1"/>
-<wire x1="11.43" y1="7.94" x2="10.16" y2="7.94" width="0.4064" layer="1"/>
+<wire x1="12.9178" y1="12.505" x2="13.335" y2="12.0878" width="0.4064" layer="1"/>
+<wire x1="13.335" y1="12.0878" x2="13.335" y2="9.525" width="0.4064" layer="1"/>
+<wire x1="13.335" y1="9.525" x2="13.02" y2="9.21" width="0.4064" layer="1"/>
+<wire x1="13.02" y1="9.21" x2="12.065" y2="9.21" width="0.4064" layer="1"/>
 </signal>
 <signal name="N$27">
 <contactref element="C4" pad="2"/>
 <contactref element="U$1" pad="16"/>
-<wire x1="12.9178" y1="13.155" x2="10.16" y2="13.155" width="0.4064" layer="1"/>
-<wire x1="10.16" y1="13.155" x2="10.16" y2="10.16" width="0.4064" layer="1"/>
-<wire x1="10.16" y1="9.84" x2="10.16" y2="10.16" width="0" layer="19" extent="1-1"/>
+<wire x1="12.9178" y1="13.155" x2="11.43" y2="13.155" width="0.4064" layer="1"/>
+<wire x1="11.43" y1="11.745" x2="12.065" y2="11.11" width="0.4064" layer="1"/>
+<wire x1="11.43" y1="13.155" x2="11.43" y2="11.745" width="0.4064" layer="1"/>
 </signal>
 <signal name="N$14">
 <contactref element="U$1" pad="14"/>
 <contactref element="C5" pad="1"/>
-<wire x1="7.62" y1="12.505" x2="7.0822" y2="12.505" width="0.4064" layer="1"/>
-<wire x1="7.62" y1="12.505" x2="7.62" y2="4.13" width="0.4064" layer="1"/>
-<wire x1="7.62" y1="4.13" x2="9.845" y2="1.905" width="0.4064" layer="1"/>
-<wire x1="9.845" y1="1.905" x2="9.845" y2="1.27" width="0.4064" layer="1"/>
+<wire x1="7.0822" y1="12.505" x2="7.62" y2="11.9672" width="0.4064" layer="1"/>
+<wire x1="7.62" y1="11.9672" x2="7.62" y2="10.475" width="0.4064" layer="1"/>
 </signal>
 <signal name="N$15">
@@
 <contactref element="JP2" pad="1"/>
 <contactref element="C5" pad="2"/>
-<wire x1="11.745" y1="1.27" x2="16.51" y2="1.27" width="0.4064" layer="1"/>
+<wire x1="7.62" y1="8.575" x2="7.62" y2="1.27" width="0.4064" layer="1"/>
+<wire x1="7.62" y1="1.27" x2="16.51" y2="1.27" width="0.4064" layer="1"/>
 </signal>
 <signal name="N$5">
 <contactref element="U$1" pad="13"/>
 <contactref element="C3" pad="2"/>
-<wire x1="6.2313" y1="12.80469375" x2="6.2313" y2="12.20530625" width="0.4064" layer="1"/>
-<wire x1="6.2313" y1="12.20530625" x2="6.35" y2="12.08660625" width="0.4064" layer="1"/>
 <wire x1="7.0822" y1="13.155" x2="6.58160625" y2="13.155" width="0.4064" layer="1"/>
-<wire x1="6.58160625" y1="13.155" x2="6.2313" y2="12.80469375" width="0.4064" layer="1"/>
-<wire x1="6.35" y1="4.13" x2="6.015" y2="3.795" width="0.4064" layer="1"/>
-<wire x1="6.35" y1="12.08660625" x2="6.35" y2="4.13" width="0.4064" layer="1"/>
+<wire x1="6.58160625" y1="13.155" x2="5.9773" y2="12.55069375" width="0.4064" layer="1"/>
+<wire x1="6.2769375" y1="4.0569375" x2="6.015" y2="3.795" width="0.4064" layer="1"/>
+<wire x1="5.9773" y1="4.356575" x2="6.2769375" y2="4.0569375" width="0.4064" layer="1"/>
+<wire x1="5.9773" y1="12.55069375" x2="5.9773" y2="4.356575" width="0.4064" layer="1"/>
 </signal>
 <signal name="N$9">
@@
 <wire x1="4.825" y1="18.355" x2="7.0822" y2="18.355" width="0.4064" layer="1"/>
 </signal>
+<signal name="PAD">
+<contactref element="U$1" pad="PAD"/>
+</signal>
 </signals>

Commit message: last update, working
Connections:
- net N$1 renamed LSS
- net N$10 renamed GLA
- net N$11 renamed GHA
- net N$12 renamed SA
- net N$13 renamed CC
- net N$14 renamed VREG
- net N$15 renamed HC
- net N$16 renamed HB
- net N$17 renamed HA
- net N$18 renamed BRAKEN
- net N$19 renamed DIR
- net N$2 renamed GLC
- net N$20 renamed ENABLE
- net N$21 renamed FAULT
- net N$22 renamed VDD
- net N$23 renamed TDEAD
- net N$24 renamed SPEED
- net N$25 renamed VBB
- net N$28 renamed VREG_GND
- net N$3 renamed GHC
- net N$4 renamed SC
- net N$5 renamed CA
- net N$6 renamed GLB
- net N$7 renamed GHB
- net N$8 renamed SB
- net N$9 renamed CB
