File: tssop28breakout/tssop28breakout.sch (EAGLE design)
At the start: 8 parts

Commit message: last version finished, pls work!
Connections:
- net GND: no longer U$1.PAD
Changed lines of the file:
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@@
 <segment>
 <pinref part="U$1" gate="G$1" pin="GND"/>
-<pinref part="U$1" gate="G$1" pin="PAD"/>
-<wire x1="22.86" y1="15.24" x2="25.4" y2="12.7" width="0.1524" layer="91"/>
-<wire x1="25.4" y1="12.7" x2="30.48" y2="12.7" width="0.1524" layer="91"/>
-<wire x1="30.48" y1="12.7" x2="30.48" y2="25.4" width="0.1524" layer="91"/>
-<wire x1="30.48" y1="25.4" x2="38.1" y2="25.4" width="0.1524" layer="91"/>
 <pinref part="JP2" gate="A" pin="2"/>
 <wire x1="38.1" y1="25.4" x2="50.8" y2="25.4" width="0.1524" layer="91"/>

Commit message: last update, working
Connections:
- net N$1 renamed LSS
- net N$10 renamed GLA
- net N$11 renamed GHA
- net N$12 renamed SA
- net N$13 renamed CC
- net N$14 renamed VREG
- net N$15 renamed HC
- net N$16 renamed HB
- net N$17 renamed HA
- net N$18 renamed BRAKEN
- net N$19 renamed DIR
- net N$2 renamed GLC
- net N$20 renamed ENABLE
- net N$21 renamed FAULT
- net N$22 renamed VDD
- net N$23 renamed TDEAD
- net N$24 renamed SPEED
- net N$25 renamed VBB
- net N$28 renamed VREG_GND
- net N$3 renamed GHC
- net N$4 renamed SC
- net N$5 renamed CA
- net N$6 renamed GLB
- net N$7 renamed GHB
- net N$8 renamed SB
- net N$9 renamed CB
Changed lines of the file:
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@@
 <?xml version="1.0" encoding="utf-8"?>
 <!DOCTYPE eagle SYSTEM "eagle.dtd">
-<eagle version="8.2.2">
+<eagle version="7.7.0">
 <drawing>
 <settings>
@@
 </busses>
 <nets>
-<net name="N$1" class="0">
+<net name="LSS" class="0">
 <segment>
 <pinref part="U$1" gate="G$1" pin="LSS"/>
@@
 </segment>
 </net>
-<net name="N$2" class="0">
+<net name="GLC" class="0">
 <segment>
 <pinref part="U$1" gate="G$1" pin="GLC"/>
@@
 </segment>
 </net>
-<net name="N$3" class="0">
+<net name="GHC" class="0">
 <segment>
 <pinref part="JP1" gate="A" pin="3"/>
@@
 </segment>
 </net>
-<net name="N$4" class="0">
+<net name="SC" class="0">
 <segment>
 <pinref part="JP1" gate="A" pin="4"/>
@@
 </segment>
 </net>
-<net name="N$6" class="0">
+<net name="GLB" class="0">
 <segment>
 <pinref part="U$1" gate="G$1" pin="GLB"/>
@@
 </segment>
 </net>
-<net name="N$7" class="0">
+<net name="GHB" class="0">
 <segment>
 <pinref part="JP1" gate="A" pin="7"/>
@@
 </segment>
 </net>
-<net name="N$8" class="0">
+<net name="SB" class="0">
 <segment>
 <pinref part="U$1" gate="G$1" pin="SB"/>
@@
 </segment>
 </net>
-<net name="N$10" class="0">
+<net name="GLA" class="0">
 <segment>
 <pinref part="U$1" gate="G$1" pin="GLA"/>
@@
 </segment>
 </net>
-<net name="N$11" class="0">
+<net name="GHA" class="0">
 <segment>
 <pinref part="JP1" gate="A" pin="11"/>
@@
 </segment>
 </net>
-<net name="N$12" class="0">
+<net name="SA" class="0">
 <segment>
 <pinref part="U$1" gate="G$1" pin="SA"/>
@@
 </segment>
 </net>
-<net name="N$14" class="0">
+<net name="VREG" class="0">
 <segment>
 <pinref part="U$1" gate="G$1" pin="VREG"/>
@@
 </segment>
 </net>
-<net name="N$15" class="0">
+<net name="HC" class="0">
 <segment>
 <pinref part="U$1" gate="G$1" pin="HC"/>
@@
 </segment>
 </net>
-<net name="N$16" class="0">
+<net name="HB" class="0">
 <segment>
 <pinref part="U$1" gate="G$1" pin="HB"/>
@@
 </segment>
 </net>
-<net name="N$17" class="0">
+<net name="HA" class="0">
 <segment>
 <pinref part="U$1" gate="G$1" pin="HA"/>
@@
 </segment>
 </net>
-<net name="N$18" class="0">
+<net name="BRAKEN" class="0">
 <segment>
 <pinref part="U$1" gate="G$1" pin="BRAKEN"/>
@@
 </segment>
 </net>
-<net name="N$19" class="0">
+<net name="DIR" class="0">
 <segment>
 <pinref part="JP2" gate="A" pin="9"/>
@@
 </segment>
 </net>
-<net name="N$20" class="0">
+<net name="ENABLE" class="0">
 <segment>
 <pinref part="U$1" gate="G$1" pin="ENABLE"/>
@@
 </segment>
 </net>
-<net name="N$21" class="0">
+<net name="FAULT" class="0">
 <segment>
 <pinref part="U$1" gate="G$1" pin="FAULT"/>
@@
 </segment>
 </net>
-<net name="N$22" class="0">
+<net name="VDD" class="0">
 <segment>
 <pinref part="U$1" gate="G$1" pin="VDD"/>
@@
 </segment>
 </net>
-<net name="N$23" class="0">
+<net name="TDEAD" class="0">
 <segment>
 <pinref part="U$1" gate="G$1" pin="TDEAD"/>
@@
 </segment>
 </net>
-<net name="N$24" class="0">
+<net name="SPEED" class="0">
 <segment>
 <pinref part="U$1" gate="G$1" pin="SPEED"/>
@@
 </segment>
 </net>
-<net name="N$25" class="0">
+<net name="VBB" class="0">
 <segment>
 <pinref part="U$1" gate="G$1" pin="VBB"/>
@@
 </segment>
 </net>
-<net name="N$28" class="0">
+<net name="VREG_GND" class="0">
 <segment>
 <pinref part="JP2" gate="A" pin="1"/>
@@
 </segment>
 </net>
-<net name="N$5" class="0">
+<net name="CA" class="0">
 <segment>
 <pinref part="U$1" gate="G$1" pin="CA"/>
@@
 </segment>
 </net>
-<net name="N$9" class="0">
+<net name="CB" class="0">
 <segment>
 <pinref part="U$1" gate="G$1" pin="CB"/>
@@
 </segment>
 </net>
-<net name="N$13" class="0">
+<net name="CC" class="0">
 <segment>
 <pinref part="U$1" gate="G$1" pin="CC"/>
