File: QEC_pcb/qec_pcb_1.brd (EAGLE design)
At the start: 50.8 x 31.1 mm, 15 parts, among them K1 68611114122

Commit message: version dos actualizada
Parts:
- R1: value (none) -> 470
- R2: value (none) -> 1k
Changed lines of the file:
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@@
 <?xml version="1.0" encoding="utf-8"?>
 <!DOCTYPE eagle SYSTEM "eagle.dtd">
-<eagle version="9.2.1">
+<eagle version="9.0.1">
 <drawing>
 <settings>
@@
 <param name="checkStop" value="0"/>
 <param name="checkValues" value="0"/>
-<param name="checkNames" value="1"/>
-<param name="checkWireStubs" value="1"/>
-<param name="checkPolygonWidth" value="0"/>
 <param name="useDiameter" value="13"/>
 <param name="maxErrors" value="50"/>
@@
 <attribute name="VALUE" x="24.765" y="7.62" size="1.27" layer="27" rot="R180"/>
 </element>
-<element name="R1" library="resistor" library_urn="urn:adsk.eagle:library:348" package="M0805" package3d_urn="urn:adsk.eagle:package:26079/1" value="" x="26.035" y="19.685" smashed="yes" rot="R270">
+<element name="R1" library="resistor" library_urn="urn:adsk.eagle:library:348" package="M0805" package3d_urn="urn:adsk.eagle:package:26079/1" value="470" x="26.035" y="19.685" smashed="yes" rot="R270">
 <attribute name="NAME" x="27.305" y="20.955" size="1.27" layer="25" rot="R270"/>
 <attribute name="VALUE" x="23.495" y="20.955" size="1.27" layer="27" rot="R270"/>
 </element>
-<element name="R2" library="resistor" library_urn="urn:adsk.eagle:library:348" package="M0805" package3d_urn="urn:adsk.eagle:package:26079/1" value="" x="22.86" y="12.7" smashed="yes" rot="R270">
+<element name="R2" library="resistor" library_urn="urn:adsk.eagle:library:348" package="M0805" package3d_urn="urn:adsk.eagle:package:26079/1" value="1k" x="22.86" y="12.7" smashed="yes" rot="R270">
 <attribute name="NAME" x="24.13" y="13.97" size="1.27" layer="25" rot="R270"/>
 <attribute name="VALUE" x="20.32" y="13.97" size="1.27" layer="27" rot="R270"/>
@@
 </signal>
 </signals>
-<mfgpreviewcolors>
-<mfgpreviewcolor name="soldermaskcolor" color="0xC8008000"/>
-<mfgpreviewcolor name="silkscreencolor" color="0xFFFEFEFE"/>
-<mfgpreviewcolor name="backgroundcolor" color="0xFF282828"/>
-<mfgpreviewcolor name="coppercolor" color="0xFFFFBF00"/>
-<mfgpreviewcolor name="substratecolor" color="0xFF786E46"/>
-</mfgpreviewcolors>
 </board>
 </drawing>
