File: QEC_pcb_v2/qec_pcb_v2.brd (EAGLE design)
At the start: 160 x 100 mm, 6 parts, among them K1 68611114122

Commit message: version dos actualizada
Parts:
- moved LED1 77.0 mm to (32.0, 6.60), turned to 90 degrees
- moved R2 67.1 mm to (26.9, 6.60)
- moved R1 55.7 mm to (29.5, 24.6), turned to 180 degrees
- moved K1 2.09 mm to (5.59, 14.5)
- moved U$1 2.09 mm to (27.2, 20.8)
- moved CTRL 2.09 mm to (50.0, 18.3)
Connections:
- removed net N$3: K1.1, U$1.6
- net DIR: now also CTRL.4; no longer CTRL.5
- net EN: now also CTRL.5; no longer CTRL.6
- net GND: now also CTRL.3; no longer CTRL.2
- net H1: now also CTRL.8; no longer CTRL.7
- net H2: now also CTRL.7; no longer CTRL.8
- net SVS: now also CTRL.2; no longer CTRL.4
- net V+: now also CTRL.6, K1.1, U$1.6; no longer CTRL.3
Routing:
- net V+: track 0.00 -> 86.2 mm
- net GND: track 0.00 -> 49.7 mm
- net H2: track 0.00 -> 47.5 mm
- net H1: track 0.00 -> 45.8 mm
- net +24V: track 0.00 -> 37.6 mm
- net N$11: track 0.00 -> 22.2 mm
- net N$12: track 0.00 -> 18.7 mm
- net SVS: track 0.00 -> 15.2 mm
- net N$5: track 0.00 -> 15.1 mm
- net N$16: track 0.00 -> 13.5 mm
- net EN: track 0.00 -> 12.9 mm
- net DIR: track 0.00 -> 10.9 mm
- net N$6: track 0.00 -> 7.30 mm
- net N$2: track 0.00 -> 5.90 mm
- net N$1: track 0.00 -> 3.08 mm
- added copper zone on layer 1, net GND
Other:
- board size 160 x 100 mm -> 53.6 x 37.5 mm
