File: QEC_pcb_v2/qec_pcb_v2.sch (EAGLE design)
At the start: 6 parts, among them K1 68611114122

Commit message: version dos actualizada
Connections:
- removed net N$3: K1.VCC, U$1.VDD
- net DIR: now also CTRL4.S; no longer CTRL5.S
- net EN: now also CTRL5.S; no longer CTRL6.S
- net GND: now also CTRL3.S; no longer CTRL2.S
- net H1: now also CTRL8.S; no longer CTRL7.S
- net H2: now also CTRL7.S; no longer CTRL8.S
- net SVS: now also CTRL2.S; no longer CTRL4.S
- net V+: now also CTRL6.S, K1.VCC, U$1.VDD; no longer CTRL3.S
Changed lines of the file:
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@@
 </segment>
 <segment>
-<pinref part="CTRL" gate="2" pin="S"/>
-<wire x1="121.92" y1="43.18" x2="116.84" y2="43.18" width="0.1524" layer="91"/>
-<label x="116.84" y="43.18" size="1.778" layer="95" rot="R180"/>
+<pinref part="CTRL" gate="3" pin="S"/>
+<wire x1="121.92" y1="40.64" x2="116.84" y2="40.64" width="0.1524" layer="91"/>
+<label x="116.84" y="40.64" size="1.778" layer="95" rot="R180"/>
 </segment>
 </net>
@@
 </segment>
 <segment>
-<pinref part="CTRL" gate="5" pin="S"/>
-<wire x1="121.92" y1="35.56" x2="116.84" y2="35.56" width="0.1524" layer="91"/>
-<label x="116.84" y="35.56" size="1.778" layer="95" rot="R180"/>
+<pinref part="CTRL" gate="4" pin="S"/>
+<wire x1="121.92" y1="38.1" x2="116.84" y2="38.1" width="0.1524" layer="91"/>
+<label x="116.84" y="38.1" size="1.778" layer="95" rot="R180"/>
 </segment>
 </net>
@@
 </segment>
 <segment>
-<pinref part="CTRL" gate="6" pin="S"/>
-<wire x1="121.92" y1="33.02" x2="116.84" y2="33.02" width="0.1524" layer="91"/>
-<label x="116.84" y="33.02" size="1.778" layer="95" rot="R180"/>
+<pinref part="CTRL" gate="5" pin="S"/>
+<wire x1="121.92" y1="35.56" x2="116.84" y2="35.56" width="0.1524" layer="91"/>
+<label x="116.84" y="35.56" size="1.778" layer="95" rot="R180"/>
 </segment>
 </net>
@@
 </segment>
 <segment>
-<pinref part="CTRL" gate="4" pin="S"/>
-<wire x1="121.92" y1="38.1" x2="116.84" y2="38.1" width="0.1524" layer="91"/>
-<label x="116.84" y="38.1" size="1.778" layer="95" rot="R180"/>
+<pinref part="CTRL" gate="2" pin="S"/>
+<wire x1="121.92" y1="43.18" x2="116.84" y2="43.18" width="0.1524" layer="91"/>
+<label x="116.84" y="43.18" size="1.778" layer="95" rot="R180"/>
 </segment>
 </net>
 <net name="V+" class="0">
 <segment>
-<pinref part="CTRL" gate="3" pin="S"/>
-<wire x1="121.92" y1="40.64" x2="116.84" y2="40.64" width="0.1524" layer="91"/>
-<label x="116.84" y="40.64" size="1.778" layer="95" rot="R180"/>
+<pinref part="U$1" gate="G$1" pin="VDD"/>
+<wire x1="50.8" y1="53.34" x2="25.4" y2="53.34" width="0.1524" layer="91"/>
+<wire x1="5.08" y1="43.18" x2="15.24" y2="43.18" width="0.1524" layer="91"/>
+<wire x1="15.24" y1="43.18" x2="25.4" y2="53.34" width="0.1524" layer="91"/>
+<pinref part="K1" gate="G$1" pin="VCC"/>
+</segment>
+<segment>
+<pinref part="CTRL" gate="6" pin="S"/>
+<wire x1="121.92" y1="33.02" x2="116.84" y2="33.02" width="0.1524" layer="91"/>
+<label x="116.84" y="33.02" size="1.778" layer="95" rot="R180"/>
 </segment>
 </net>
@@
 </segment>
 <segment>
-<pinref part="CTRL" gate="8" pin="S"/>
-<wire x1="121.92" y1="27.94" x2="116.84" y2="27.94" width="0.1524" layer="91"/>
-<label x="116.84" y="27.94" size="1.778" layer="95" rot="R180"/>
+<pinref part="CTRL" gate="7" pin="S"/>
+<wire x1="121.92" y1="30.48" x2="116.84" y2="30.48" width="0.1524" layer="91"/>
+<label x="116.84" y="30.48" size="1.778" layer="95" rot="R180"/>
 </segment>
 </net>
@@
 </segment>
 <segment>
-<pinref part="CTRL" gate="7" pin="S"/>
-<wire x1="121.92" y1="30.48" x2="116.84" y2="30.48" width="0.1524" layer="91"/>
-<label x="116.84" y="30.48" size="1.778" layer="95" rot="R180"/>
+<pinref part="CTRL" gate="8" pin="S"/>
+<wire x1="121.92" y1="27.94" x2="116.84" y2="27.94" width="0.1524" layer="91"/>
+<label x="116.84" y="27.94" size="1.778" layer="95" rot="R180"/>
 </segment>
 </net>
@@
 </segment>
 </net>
-<net name="N$3" class="0">
-<segment>
-<pinref part="U$1" gate="G$1" pin="VDD"/>
-<wire x1="50.8" y1="53.34" x2="25.4" y2="53.34" width="0.1524" layer="91"/>
-<wire x1="5.08" y1="43.18" x2="15.24" y2="43.18" width="0.1524" layer="91"/>
-<wire x1="15.24" y1="43.18" x2="25.4" y2="53.34" width="0.1524" layer="91"/>
-<pinref part="K1" gate="G$1" pin="VCC"/>
-</segment>
-</net>
