File: QEC_pcb_v4/qec_pcb_v4.sch (EAGLE design)
At the start: 6 parts, among them K1 68611114122

Commit message: ultima version motor controller
Parts:
- renumbered K1 to MOTOR, U$1 to DEC
Changed lines of the file:
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@@
 <?xml version="1.0" encoding="utf-8"?>
 <!DOCTYPE eagle SYSTEM "eagle.dtd">
-<eagle version="9.4.2">
+<eagle version="9.6.1">
 <drawing>
 <settings>
@@
 </classes>
 <parts>
-<part name="U$1" library="dedo" deviceset="1-Q-EC" device="1-Q-EC-SMD" value="1-Q-EC1-Q-EC-SMD"/>
+<part name="DEC" library="dedo" deviceset="1-Q-EC" device="1-Q-EC-SMD" value="1-Q-EC1-Q-EC-SMD"/>
 <part name="R1" library="resistor" library_urn="urn:adsk.eagle:library:348" deviceset="R-US_" device="M0805" package3d_urn="urn:adsk.eagle:package:23556/1" value="470"/>
 <part name="R2" library="resistor" library_urn="urn:adsk.eagle:library:348" deviceset="R-US_" device="M0805" package3d_urn="urn:adsk.eagle:package:23556/1" value="1k"/>
@@
 <part name="P+1" library="supply1" library_urn="urn:adsk.eagle:library:371" deviceset="+24V" device=""/>
 <part name="GND2" library="supply1" library_urn="urn:adsk.eagle:library:371" deviceset="GND" device=""/>
-<part name="K1" library="dedo" deviceset="68611114122" device=""/>
+<part name="MOTOR" library="dedo" deviceset="68611114122" device=""/>
 <part name="CTRL" library="dedo" deviceset="JST8" device=""/>
 <part name="GND3" library="supply1" library_urn="urn:adsk.eagle:library:371" deviceset="GND" device=""/>
@@
 </plain>
 <instances>
-<instance part="U$1" gate="G$1" x="93.98" y="53.34" smashed="yes"/>
+<instance part="DEC" gate="G$1" x="93.98" y="53.34" smashed="yes"/>
 <instance part="R1" gate="G$1" x="99.06" y="63.5" smashed="yes">
 <attribute name="NAME" x="95.25" y="64.9986" size="1.778" layer="95"/>
@@
 <attribute name="VALUE" x="38.1" y="22.86" size="1.778" layer="96"/>
 </instance>
-<instance part="K1" gate="G$1" x="20.32" y="48.26" smashed="yes"/>
+<instance part="MOTOR" gate="G$1" x="20.32" y="48.26" smashed="yes"/>
 <instance part="CTRL" gate="1" x="124.46" y="40.64" smashed="yes">
 <attribute name="NAME" x="127" y="39.878" size="1.524" layer="95"/>
@@
 </segment>
 <segment>
-<pinref part="U$1" gate="G$1" pin="GND"/>
+<pinref part="DEC" gate="G$1" pin="GND"/>
 <pinref part="GND2" gate="1" pin="GND"/>
 <wire x1="50.8" y1="55.88" x2="40.64" y2="55.88" width="0.1524" layer="91"/>
@@
 <wire x1="12.7" y1="53.34" x2="10.16" y2="53.34" width="0.1524" layer="91"/>
 <junction x="40.64" y="55.88"/>
-<pinref part="K1" gate="G$1" pin="GND"/>
+<pinref part="MOTOR" gate="G$1" pin="GND"/>
 <wire x1="10.16" y1="53.34" x2="7.62" y2="53.34" width="0.1524" layer="91"/>
 <wire x1="7.62" y1="53.34" x2="5.08" y2="53.34" width="0.1524" layer="91"/>
@@
 <segment>
 <pinref part="R1" gate="G$1" pin="2"/>
-<pinref part="U$1" gate="G$1" pin="GND2"/>
+<pinref part="DEC" gate="G$1" pin="GND2"/>
 <wire x1="104.14" y1="63.5" x2="104.14" y2="60.96" width="0.1524" layer="91"/>
 <wire x1="104.14" y1="60.96" x2="81.28" y2="60.96" width="0.1524" layer="91"/>
@@
 <pinref part="GND3" gate="1" pin="GND"/>
 <junction x="114.3" y="50.8"/>
-<pinref part="U$1" gate="G$1" pin="DN2"/>
+<pinref part="DEC" gate="G$1" pin="DN2"/>
 <wire x1="81.28" y1="53.34" x2="114.3" y2="53.34" width="0.1524" layer="91"/>
-<pinref part="U$1" gate="G$1" pin="DN1"/>
+<pinref part="DEC" gate="G$1" pin="DN1"/>
 <wire x1="81.28" y1="50.8" x2="114.3" y2="50.8" width="0.1524" layer="91"/>
 </segment>
@@
 <net name="N$2" class="0">
 <segment>
-<pinref part="U$1" gate="G$1" pin="RDY"/>
+<pinref part="DEC" gate="G$1" pin="RDY"/>
 <pinref part="LED1" gate="G$1" pin="A"/>
 <wire x1="81.28" y1="48.26" x2="88.9" y2="48.26" width="0.1524" layer="91"/>
@@
 <segment>
 <pinref part="R1" gate="G$1" pin="1"/>
-<pinref part="U$1" gate="G$1" pin="SCL"/>
+<pinref part="DEC" gate="G$1" pin="SCL"/>
 <wire x1="93.98" y1="63.5" x2="81.28" y2="63.5" width="0.1524" layer="91"/>
 </segment>
@@
 <net name="DIR" class="0">
 <segment>
-<pinref part="U$1" gate="G$1" pin="DIR"/>
+<pinref part="DEC" gate="G$1" pin="DIR"/>
 <wire x1="81.28" y1="58.42" x2="106.68" y2="58.42" width="0.1524" layer="91"/>
 <wire x1="106.68" y1="58.42" x2="106.68" y2="71.12" width="0.1524" layer="91"/>
@@
 <net name="EN" class="0">
 <segment>
-<pinref part="U$1" gate="G$1" pin="EN"/>
+<pinref part="DEC" gate="G$1" pin="EN"/>
 <wire x1="81.28" y1="55.88" x2="109.22" y2="55.88" width="0.1524" layer="91"/>
 <wire x1="109.22" y1="55.88" x2="109.22" y2="68.58" width="0.1524" layer="91"/>
@@
 <net name="SVS" class="0">
 <segment>
-<pinref part="U$1" gate="G$1" pin="SVS"/>
+<pinref part="DEC" gate="G$1" pin="SVS"/>
 <wire x1="81.28" y1="66.04" x2="104.14" y2="66.04" width="0.1524" layer="91"/>
 <wire x1="104.14" y1="66.04" x2="104.14" y2="73.66" width="0.1524" layer="91"/>
@@
 <net name="V+" class="0">
 <segment>
-<pinref part="U$1" gate="G$1" pin="VDD"/>
+<pinref part="DEC" gate="G$1" pin="VDD"/>
 <wire x1="50.8" y1="53.34" x2="25.4" y2="53.34" width="0.1524" layer="91"/>
 <wire x1="5.08" y1="43.18" x2="15.24" y2="43.18" width="0.1524" layer="91"/>
 <wire x1="15.24" y1="43.18" x2="25.4" y2="53.34" width="0.1524" layer="91"/>
-<pinref part="K1" gate="G$1" pin="VCC"/>
+<pinref part="MOTOR" gate="G$1" pin="VCC"/>
 </segment>
 <segment>
@@
 <net name="+24V" class="0">
 <segment>
-<pinref part="U$1" gate="G$1" pin="VCC"/>
+<pinref part="DEC" gate="G$1" pin="VCC"/>
 <wire x1="50.8" y1="58.42" x2="40.64" y2="58.42" width="0.1524" layer="91"/>
 <pinref part="P+1" gate="1" pin="+24V"/>
@@
 <net name="H2" class="0">
 <segment>
-<pinref part="U$1" gate="G$1" pin="H2"/>
+<pinref part="DEC" gate="G$1" pin="H2"/>
 <wire x1="5.08" y1="50.8" x2="12.7" y2="50.8" width="0.1524" layer="91"/>
 <wire x1="12.7" y1="50.8" x2="15.24" y2="48.26" width="0.1524" layer="91"/>
 <wire x1="15.24" y1="48.26" x2="50.8" y2="48.26" width="0.1524" layer="91"/>
-<pinref part="K1" gate="G$1" pin="H2"/>
+<pinref part="MOTOR" gate="G$1" pin="H2"/>
 <label x="38.1" y="48.26" size="1.778" layer="95" rot="R180" xref="yes"/>
 </segment>
@@
 <net name="N$5" class="0">
 <segment>
-<pinref part="U$1" gate="G$1" pin="W1"/>
+<pinref part="DEC" gate="G$1" pin="W1"/>
 <wire x1="50.8" y1="66.04" x2="15.24" y2="66.04" width="0.1524" layer="91"/>
 <wire x1="15.24" y1="66.04" x2="10.16" y2="60.96" width="0.1524" layer="91"/>
-<pinref part="K1" gate="G$1" pin="W1"/>
+<pinref part="MOTOR" gate="G$1" pin="W1"/>
 <wire x1="10.16" y1="60.96" x2="5.08" y2="60.96" width="0.1524" layer="91"/>
 </segment>
@@
 <net name="N$11" class="0">
 <segment>
-<pinref part="U$1" gate="G$1" pin="W2"/>
+<pinref part="DEC" gate="G$1" pin="W2"/>
 <wire x1="50.8" y1="63.5" x2="15.24" y2="63.5" width="0.1524" layer="91"/>
 <wire x1="15.24" y1="63.5" x2="10.16" y2="58.42" width="0.1524" layer="91"/>
-<pinref part="K1" gate="G$1" pin="W2"/>
+<pinref part="MOTOR" gate="G$1" pin="W2"/>
 <wire x1="10.16" y1="58.42" x2="5.08" y2="58.42" width="0.1524" layer="91"/>
 </segment>
@@
 <net name="N$12" class="0">
 <segment>
-<pinref part="U$1" gate="G$1" pin="W3"/>
+<pinref part="DEC" gate="G$1" pin="W3"/>
 <wire x1="50.8" y1="60.96" x2="15.24" y2="60.96" width="0.1524" layer="91"/>
 <wire x1="15.24" y1="60.96" x2="10.16" y2="55.88" width="0.1524" layer="91"/>
-<pinref part="K1" gate="G$1" pin="W3"/>
+<pinref part="MOTOR" gate="G$1" pin="W3"/>
 <wire x1="10.16" y1="55.88" x2="5.08" y2="55.88" width="0.1524" layer="91"/>
 </segment>
@@
 <net name="H1" class="0">
 <segment>
-<pinref part="U$1" gate="G$1" pin="H1"/>
+<pinref part="DEC" gate="G$1" pin="H1"/>
 <wire x1="50.8" y1="50.8" x2="15.24" y2="50.8" width="0.1524" layer="91"/>
 <wire x1="15.24" y1="50.8" x2="12.7" y2="48.26" width="0.1524" layer="91"/>
 <wire x1="12.7" y1="48.26" x2="10.16" y2="48.26" width="0.1524" layer="91"/>
-<pinref part="K1" gate="G$1" pin="H1"/>
+<pinref part="MOTOR" gate="G$1" pin="H1"/>
 <wire x1="10.16" y1="48.26" x2="7.62" y2="48.26" width="0.1524" layer="91"/>
 <wire x1="7.62" y1="48.26" x2="5.08" y2="48.26" width="0.1524" layer="91"/>
@@
 <net name="N$16" class="0">
 <segment>
-<pinref part="U$1" gate="G$1" pin="H3"/>
+<pinref part="DEC" gate="G$1" pin="H3"/>
 <wire x1="50.8" y1="45.72" x2="10.16" y2="45.72" width="0.1524" layer="91"/>
-<pinref part="K1" gate="G$1" pin="H3"/>
+<pinref part="MOTOR" gate="G$1" pin="H3"/>
 <wire x1="10.16" y1="45.72" x2="7.62" y2="45.72" width="0.1524" layer="91"/>
 <wire x1="7.62" y1="45.72" x2="5.08" y2="45.72" width="0.1524" layer="91"/>

Commit message: update directories
Connections:
- net N$16 renamed H3
Changed lines of the file:
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@@
 </segment>
 </net>
-<net name="N$16" class="0">
+<net name="H3" class="0">
 <segment>
 <pinref part="DEC" gate="G$1" pin="H3"/>
